Commit message: keyboard teleop

File: description/lemower.xacro (robot description, xacro)
@@ -79,10 +79,8 @@
         </xacro:inertial_box>
     </link>
-    <joint name="robot_base_to_bras_decoupe" type="revolute">
+    <joint name="robot_base_to_bras_decoupe" type="fixed">
         <parent link="robot_base"/>
         <child link="bras decoupe"/>
         <origin xyz="0.31 0 0.03" rpy="0 0 0"/>
-        <limit effort="1000.0" lower="-0.548" upper="0.548" velocity="0.5"/>
-        <axis xyz="0 1 0"/>
     </joint>
     <link name="bras decoupe">
@@ -104,10 +102,8 @@
         </xacro:inertial_box>
     </link>
-    <joint name="bras_decoupe_to_decoupe" type="revolute">
+    <joint name="bras_decoupe_to_decoupe" type="fixed">
         <parent link="bras decoupe"/>
         <child link="decoupe"/>
-        <axis xyz="0 1 0"/>
         <origin xyz="0.05 0 0" rpy="0 0 0"/>
-        <limit effort="1000.0" lower="-0.548" upper="0.548" velocity="0.5"/>
     </joint>
     <link name="decoupe">

File: description/lemower_gazebo.xacro (robot description, xacro)
@@ -62,8 +62,14 @@
             <topic>/joint_states</topic> <!-- Nom du topic côté Gazebo -->
             <update_rate>30</update_rate>
-            <joint_name>robot_base_to_bras_decoupe</joint_name>
-            <joint_name>bras_decoupe_to_decoupe</joint_name>
             <joint_name>base_to_roue_arriere_gauche</joint_name>
             <joint_name>base_to_roue_arriere_droite</joint_name>
+        </plugin>
+        <plugin filename="gz-sim-odometry-publisher-system" name="gz::sim::systems::OdometryPublisher">
+	    <odom_frame>odom</odom_frame>
+	    <robot_base_frame>base_link</robot_base_frame>
+            <odom_publish_frequency>50</odom_publish_frequency>
+            <odom_topic>/odom</odom_topic>
+            <tf_topic>/tf</tf_topic>
+            <dimensions>2</dimensions>
         </plugin>
     </gazebo>
@@ -74,16 +80,24 @@
     <!-- Here's an example message to publish to test it:
             ros2 topic pub -1 /set_joint_trajectory trajectory_msgs/msg/JointTrajectory  '{header: {frame_id: world}, joint_names: [slider_joint, arm_joint], points: [  {positions: {0.8,0.6}} ]}' -->
-    <gazebo>
-        <plugin filename="gz-sim-joint-trajectory-controller-system" name="gz::sim::systems::JointTrajectoryController">
-            <topic>/model/lemower/joint_trajectory</topic>
-        </plugin>
+    <!-- Gazebo Parameters -->
+    <gazebo reference="Roue arrière gauche">
+        <mu1>1.0</mu1>
+        <mu2>1.0</mu2>
+    </gazebo>
+    <gazebo reference="Roue arrière droite">
+        <mu1>1.0</mu1>
+        <mu2>1.0</mu2>
+    </gazebo>
+    <gazebo reference="base_link">
+        <mu1>1.0</mu1>
+        <mu2>1.0</mu2>
     </gazebo>
     <gazebo reference="Roue avant droite">
-        <mu value="0"/>
-        <mu2 value="1"/>
+        <mu1>0.00001</mu1>
+        <mu2>0.00001</mu2>
     </gazebo>
     <gazebo reference="Roue avant gauche">
-        <mu value="0"/>
-        <mu2 value="1"/>
+        <mu1>0.00001</mu1>
+        <mu2>0.00001</mu2>
     </gazebo>
 </robot>

Commit message: Manage xacro segregation and lidar

File: description/lemower.xacro (robot description, xacro)
@@ -4,267 +4,8 @@
     <!-- This will include all the contents of example_include.xacro first. Go check it out! -->
     <xacro:include filename="lemower_include.xacro" />
-    <!-- Then base link is aligned with the wheels
-           Former position = <origin xyz="-0.07 -0.095 -0.039" rpy="0 1.5708 0"/>
-     -->
-    <link name="base_link">
-    </link>
-    <!-- Lien entre base et robot_base l'origine de robot_base est arrière centre bas -->
-    <joint name="robot_base_joint" type="fixed">
-        <parent link="base_link"/>
-        <child link="robot_base"/>
-        <origin xyz="-0.065 0 0.029" rpy="0 0 0"/>
-    </joint>
-    <link name="robot_base">
-        <visual>
-            <geometry>
-                <box size="0.32 0.2 0.04"/>
-            </geometry>
-            <material name="blue"/>
-            <origin xyz="0.16 0 0.02" rpy="0 0 0"/>
-        </visual>
-        <collision>
-            <geometry>
-                <box size="0.32 0.2 0.04"/>
-            </geometry>
-            <origin xyz="0.16 0 0.02" rpy="0 0 0"/>
-        </collision>
-        <xacro:inertial_box mass="1.5" x="0.18" y="0.2" z="0.04">
-            <origin xyz="0.09 0 0.02" rpy="0 0 0"/>
-        </xacro:inertial_box>
-    </link>
-    <joint name="base_to_elec" type="fixed">
-        <parent link="robot_base"/>
-        <child link="electronics"/>
-        <origin xyz="0 0 0.04" rpy="0 0 0"/>
-    </joint>
-    <link name="electronics">
-        <visual>
-            <geometry>
-                <box size="0.15 0.2 0.04"/>
-            </geometry>
-            <origin xyz="0.075 0 0.02" rpy="0 0 0"/>
-            <material name="blue"/>
-        </visual>
-        <collision>
-            <geometry>
-                <box size="0.15 0.2 0.04"/>
-            </geometry>
-            <origin xyz="0.075 0 0.02" rpy="0 0 0"/>
-        </collision>
-        <xacro:inertial_box mass="0.4" x="0.15" y="0.2" z="0.04">
-            <origin xyz="0.075 0 0.02" rpy="0 0 0"/>
-        </xacro:inertial_box>
-    </link>
-    <joint name="elec_to_lidar" type="fixed">
-        <parent link="electronics"/>
-        <child link="lidar"/>
-        <origin xyz="0.075 0 0.04" rpy="0 0 0"/>
-    </joint>
-    <link name="lidar">
-        <visual>
-            <geometry>
-                <box size="0.06 0.05 0.03"/>
-            </geometry>
-            <origin xyz="0 0 0.015" rpy="0 0 0"/>
-            <material name="black"/>
-        </visual>
-        <collision>
-            <origin xyz="0 0 0.015" rpy="0 0 0"/>
-            <geometry>
-                <box size="0.06 0.05 0.03"/>
-            </geometry>
-        </collision>
-        <xacro:inertial_box mass="0.1" x="0.06" y="0.05" z="0.03">
-            <origin xyz="0 0 0.015" rpy="0 0 0"/>
-        </xacro:inertial_box>
-    </link>
-    <joint name="robot_base_to_bras_decoupe" type="fixed">
-        <parent link="robot_base"/>
-        <child link="bras decoupe"/>
-        <origin xyz="0.31 0 0.03" rpy="0 0 0"/>
-    </joint>
-    <link name="bras decoupe">
-        <visual>
-            <geometry>
-                <box size="0.06 0.003 0.01"/>
-            </geometry>
-            <origin xyz="0.028 0 0.005" rpy="0 0 0"/>
-            <material name="blue"/>
-        </visual>
-        <collision>
-            <origin xyz="0.028 0 0.005" rpy="0 0 0"/>
-            <geometry>
-                <box size="0.06 0.003 0.01"/>
-            </geometry>
-        </collision>
-        <xacro:inertial_box mass="0.05" x="0.06" y="0.003" z="0.01">
-            <origin xyz="0.03 0.0015 0.005" rpy="0 0 0"/>
-        </xacro:inertial_box>
-    </link>
-    <joint name="bras_decoupe_to_decoupe" type="fixed">
-        <parent link="bras decoupe"/>
-        <child link="decoupe"/>
-        <origin xyz="0.05 0 0" rpy="0 0 0"/>
-    </joint>
-    <link name="decoupe">
-        <visual>
-            <geometry>
-                <box size="0.1 0.3 0.06"/>
-            </geometry>
-            <origin xyz="0.045 0 0" rpy="0 0 0"/>
-            <material name="red"/>
-        </visual>
-        <collision>
-            <origin xyz="0.045 0 0" rpy="0 0 0"/>
-            <geometry>
-                <box size="0.1 0.3 0.06"/>
-            </geometry>
-        </collision>
-        <xacro:inertial_box mass="0.5" x="0.1" y="0.3" z="0.06">
-            <origin xyz="0.05 0 0" rpy="0 0 0"/>
-        </xacro:inertial_box>
-    </link>
-    <joint name="base_to_motor_gauche" type="fixed">
-        <parent link="base_link"/>
-        <child link="motor gauche"/>
-        <origin xyz="0 0.07 0.0075" rpy="0 0 0"/>
-    </joint>
-    <link name="motor gauche">
-        <visual>
-            <origin xyz="0 0 0" rpy="1.5708 0 0"/>
-            <geometry>
-                <cylinder length="0.057" radius="0.0185"/>
-            </geometry>
-            <material name="red"/>
-        </visual>
-        <collision>
-            <origin xyz="0 0 0" rpy="1.5708 0 0"/>
-            <geometry>
-                <cylinder length="0.057" radius="0.0185"/>
-            </geometry>
-        </collision>
-        <xacro:inertial_cylinder mass="0.15" length="0.057" radius="0.0185">
-            <origin xyz="0 0 0" rpy="0 0 0"/>
-        </xacro:inertial_cylinder>
-    </link>
-    <joint name="base_to_motor_droite" type="fixed">
-        <parent link="base_link"/>
-        <child link="motor droite"/>
-        <origin xyz="0 -0.07 0.0075" rpy="0 0 0"/>
-    </joint>
-    <link name="motor droite">
-        <visual>
-            <origin xyz="0 0 0" rpy="1.5708 0 0"/>
-            <geometry>
-                <cylinder length="0.057" radius="0.0185"/>
-            </geometry>
-            <material name="red"/>
-        </visual>
-        <collision>
-            <origin xyz="0 0 0" rpy="1.5708 0 0"/>
-            <geometry>
-                <cylinder length="0.057" radius="0.0185"/>
-            </geometry>
-        </collision>
-        <xacro:inertial_cylinder mass="0.15" length="0.057" radius="0.0185">
-            <origin xyz="0 0 0" rpy="0 0 0"/>
-        </xacro:inertial_cylinder>
-    </link>
-    <joint name="base_to_roue_arriere_gauche" type="continuous">
-        <parent link="base_link"/>
-        <child link="Roue arrière gauche"/>
-        <origin xyz="0 0.125 0" rpy="-${pi/2} 0 0"/>
-        <axis xyz="0 0 1"/>
-        <limit effort="0.05" velocity="10.0"/>
-    </joint>
-    <link name="Roue arrière gauche">
-        <visual>
-            <origin xyz="0 0 0" rpy="0 0 0"/>
-            <geometry>
-                <cylinder length="0.045" radius="0.048"/>
-            </geometry>
-            <material name="green"/>
-        </visual>
-        <collision>
-            <origin xyz="0 0 0" rpy="0 0 0"/>
-            <geometry>
-                <sphere radius="0.048" />
-            </geometry>
-        </collision>
-        <xacro:inertial_cylinder mass="0.2" length="0.045" radius="0.048">
-            <origin xyz="0 0 0" rpy="0 0 0"/>
-        </xacro:inertial_cylinder>
-    </link>
-    <joint name="base_to_roue_arriere_droite" type="continuous">
-        <parent link="base_link"/>
-        <child link="Roue arrière droite"/>
-        <origin xyz="0 -0.125 0" rpy="${pi/2} 0 0"/>
-        <limit effort="0.05" velocity="10.0"/>
-        <axis xyz="0 0 -1"/>
-    </joint>
-    <link name="Roue arrière droite">
-        <visual>
-            <origin xyz="0 0 0" rpy="0 0 0"/>
-            <geometry>
-                <cylinder length="0.045" radius="0.048"/>
-            </geometry>
-            <material name="green"/>
-        </visual>
-        <collision>
-            <origin xyz="0 0 0" rpy="0 0 0"/>
-            <geometry>
-                <sphere radius="0.048" />
-            </geometry>
-        </collision>
-        <xacro:inertial_cylinder mass="0.2" length="0.045" radius="0.048">
-            <origin xyz="0 0 0" rpy="0 0 0"/>
-        </xacro:inertial_cylinder>
-    </link>
-    <joint name="robot_base_to_roue_avant_gauche" type="fixed">
-        <parent link="robot_base"/>
-        <child link="Roue avant gauche"/>
-        <origin xyz="0.268 0.125 -0.043" rpy="-${pi/2} 0 0"/>
-    </joint>
-    <link name="Roue avant gauche">
-        <visual>
-            <origin xyz="0 0 0" rpy="0 0 0"/>
-            <geometry>
-                <cylinder length="0.045" radius="0.034"/>
-            </geometry>
-            <material name="green"/>
-        </visual>
-        <collision>
-            <origin xyz="0 0 0" rpy="0 0 0"/>
-            <geometry>
-                <sphere radius="0.034" />
-            </geometry>
-        </collision>
-        <xacro:inertial_cylinder mass="0.2" length="0.045" radius="0.034">
-            <origin xyz="0 0 0" rpy="0 0 0"/>
-        </xacro:inertial_cylinder>
-    </link>
-    <joint name="robot_base_to_roue_avant_droite" type="fixed">
-        <parent link="robot_base"/>
-        <child link="Roue avant droite"/>
-        <origin xyz="0.268 -0.125 -0.043" rpy="${pi/2} 0 0"/>
-    </joint>
-    <link name="Roue avant droite">
-        <visual>
-            <origin xyz="0 0 0" rpy="0 0 0"/>
-            <geometry>
-                <cylinder length="0.045" radius="0.034"/>
-            </geometry>
-            <material name="green"/>
-        </visual>
-        <collision>
-            <origin xyz="0 0 0" rpy="0 0 0"/>
-            <geometry>
-                <sphere radius="0.034" />
-            </geometry>
-        </collision>
-        <xacro:inertial_cylinder mass="0.2" length="0.045" radius="0.034">
-            <origin xyz="0 0 0" rpy="0 0 0"/>
-        </xacro:inertial_cylinder>
-    </link>
+    <!-- This file is the description of the robot -->
+    <xacro:include filename="lemower_core.xacro" />
     <xacro:include filename="lemower_gazebo.xacro" />
+    <xacro:include filename="ros2_control.xacro"/>
+    <!-- <xacro:include filename="lemower_gz_control.xacro" /> -->
 </robot>

File: description/lemower_core.xacro (robot description, xacro)
@@ -2,6 +2,4 @@
 <!-- Description of the LEMOWER robot with XACRO to avoid repeating data -->
 <robot xmlns:xacro="http://www.ros.org/wiki/xacro"  name="lemower">
-    <!-- This will include all the contents of example_include.xacro first. Go check it out! -->
-    <xacro:include filename="lemower_include.xacro" />
     <!-- Then base link is aligned with the wheels
            Former position = <origin xyz="-0.07 -0.095 -0.039" rpy="0 1.5708 0"/>
@@ -9,4 +7,8 @@
     <link name="base_link">
     </link>
+    <gazebo reference="base_link">
+        <mu1>1.0</mu1>
+        <mu2>1.0</mu2>
+    </gazebo>
     <!-- Lien entre base et robot_base l'origine de robot_base est arrière centre bas -->
     <joint name="robot_base_joint" type="fixed">
@@ -33,4 +35,7 @@
         </xacro:inertial_box>
     </link>
+    <gazebo reference="robot_base">
+        <material>Gazebo/Blue</material>
+    </gazebo>
     <joint name="base_to_elec" type="fixed">
         <parent link="robot_base"/>
@@ -56,4 +61,7 @@
         </xacro:inertial_box>
     </link>
+    <gazebo reference="electronics">
+        <material>Gazebo/Blue</material>
+    </gazebo>
     <joint name="elec_to_lidar" type="fixed">
         <parent link="electronics"/>
@@ -64,5 +72,5 @@
         <visual>
             <geometry>
-                <box size="0.06 0.05 0.03"/>
+                <cylinder radius="0.05" length="0.04"/>
             </geometry>
             <origin xyz="0 0 0.015" rpy="0 0 0"/>
@@ -72,17 +80,18 @@
             <origin xyz="0 0 0.015" rpy="0 0 0"/>
             <geometry>
-                <box size="0.06 0.05 0.03"/>
-            </geometry>
-        </collision>
-        <xacro:inertial_box mass="0.1" x="0.06" y="0.05" z="0.03">
+                <cylinder radius="0.05" length="0.04"/>
+            </geometry>
+        </collision>
+        <xacro:inertial_cylinder mass="0.1" length="0.04" radius="0.05">
             <origin xyz="0 0 0.015" rpy="0 0 0"/>
-        </xacro:inertial_box>
-    </link>
-    <joint name="robot_base_to_bras_decoupe" type="revolute">
+        </xacro:inertial_cylinder>
+    </link>
+    <gazebo reference="lidar">
+        <material>Gazebo/Black</material>
+    </gazebo>
+    <joint name="robot_base_to_bras_decoupe" type="fixed">
         <parent link="robot_base"/>
         <child link="bras decoupe"/>
         <origin xyz="0.31 0 0.03" rpy="0 0 0"/>
-        <limit effort="1000.0" lower="-0.548" upper="0.548" velocity="0.5"/>
-        <axis xyz="0 1 0"/>
     </joint>
     <link name="bras decoupe">
@@ -104,10 +113,11 @@
         </xacro:inertial_box>
     </link>
-    <joint name="bras_decoupe_to_decoupe" type="revolute">
+    <gazebo reference="bras decoupe">
+        <material>Gazebo/Blue</material>
+    </gazebo>
+    <joint name="bras_decoupe_to_decoupe" type="fixed">
         <parent link="bras decoupe"/>
         <child link="decoupe"/>
-        <axis xyz="0 1 0"/>
         <origin xyz="0.05 0 0" rpy="0 0 0"/>
-        <limit effort="1000.0" lower="-0.548" upper="0.548" velocity="0.5"/>
     </joint>
     <link name="decoupe">
@@ -129,4 +139,7 @@
         </xacro:inertial_box>
     </link>
+    <gazebo reference="decoupe">
+        <material>Gazebo/Red</material>
+    </gazebo>
     <joint name="base_to_motor_gauche" type="fixed">
         <parent link="base_link"/>
@@ -152,4 +165,7 @@
         </xacro:inertial_cylinder>
     </link>
+    <gazebo reference="motor gauche">
+        <material>Gazebo/Red</material>
+    </gazebo>
     <joint name="base_to_motor_droite" type="fixed">
         <parent link="base_link"/>
@@ -175,4 +191,7 @@
         </xacro:inertial_cylinder>
     </link>
+    <gazebo reference="motor droite">
+        <material>Gazebo/Red</material>
+    </gazebo>
     <joint name="base_to_roue_arriere_gauche" type="continuous">
         <parent link="base_link"/>
@@ -200,4 +219,9 @@
         </xacro:inertial_cylinder>
     </link>
+    <gazebo reference="Roue arrière gauche">
+        <material>Gazebo/Green</material>
+        <mu1>1.0</mu1>
+        <mu2>1.0</mu2>
+    </gazebo>
     <joint name="base_to_roue_arriere_droite" type="continuous">
         <parent link="base_link"/>
@@ -225,4 +249,9 @@
         </xacro:inertial_cylinder>
     </link>
+    <gazebo reference="Roue arrière droite">
+        <material>Gazebo/Green</material>
+        <mu1>1.0</mu1>
+        <mu2>1.0</mu2>
+    </gazebo>
     <joint name="robot_base_to_roue_avant_gauche" type="fixed">
         <parent link="robot_base"/>
@@ -248,4 +277,9 @@
         </xacro:inertial_cylinder>
     </link>
+    <gazebo reference="Roue avant gauche">
+        <material>Gazebo/Green</material>
+        <mu1>0.00001</mu1>
+        <mu2>0.00001</mu2>
+    </gazebo>
     <joint name="robot_base_to_roue_avant_droite" type="fixed">
         <parent link="robot_base"/>
@@ -271,4 +305,8 @@
         </xacro:inertial_cylinder>
     </link>
-    <xacro:include filename="lemower_gazebo.xacro" />
+    <gazebo reference="Roue avant droite">
+        <material>Gazebo/Green</material>
+        <mu1>0.00001</mu1>
+        <mu2>0.00001</mu2>
+    </gazebo>
 </robot>

File: description/lemower_gazebo.xacro (robot description, xacro)
@@ -6,53 +6,4 @@
     <!-- Gazebo is unable to use the same <material> tags that are already in the URDF (that RViz uses). -->
     <!-- Instead, we need to add gazebo tags for our links that refer to Gazebo materials -->
-    <gazebo reference="robot_base">
-        <material>Gazebo/Blue</material>
-    </gazebo>
-    <gazebo reference="electronics">
-        <material>Gazebo/Blue</material>
-    </gazebo>
-    <gazebo reference="lidar">
-        <material>Gazebo/Black</material>
-    </gazebo>
-    <gazebo reference="bras decoupe">
-        <material>Gazebo/Blue</material>
-    </gazebo>
-    <gazebo reference="decoupe">
-        <material>Gazebo/Red</material>
-    </gazebo>
-    <gazebo reference="motor gauche">
-        <material>Gazebo/Red</material>
-    </gazebo>
-    <gazebo reference="motor droite">
-        <material>Gazebo/Red</material>
-    </gazebo>
-    <gazebo reference="Roue arrière gauche">
-        <material>Gazebo/Green</material>
-    </gazebo>
-    <gazebo reference="Roue arrière droite">
-        <material>Gazebo/Green</material>
-    </gazebo>
-    <gazebo reference="Roue avant gauche">
-        <material>Gazebo/Green</material>
-    </gazebo>
-    <gazebo reference="Roue avant droite">
-        <material>Gazebo/Green</material>
-    </gazebo>
-    <gazebo>
-          <plugin name="gz::sim::systems::DiffDrive" filename="gz-sim-diff-drive-system">
-            <!-- Wheel Information -->
-            <left_joint>base_to_roue_arriere_gauche</left_joint>
-            <right_joint>base_to_roue_arriere_droite</right_joint>
-            <wheel_separation>0.223</wheel_separation>
-            <wheel_radius>0.048</wheel_radius>
-            <!-- Input -->
-            <topic>cmd_vel</topic>
-            <!-- Output -->
-            <frame_id>odom</frame_id>
-            <child_frame_id>base_link</child_frame_id>
-            <odom_topic>odom</odom_topic>
-            <tf_topic>tf</tf_topic>
-        </plugin>
-    </gazebo>
     <!-- Gazebo requires the use of plugins to interact with other systems such as ROS. -->
     <!-- This plugin will publish the joint_states for the selected joints
@@ -74,30 +25,36 @@
         </plugin>
     </gazebo>
-    <!-- This plugin will read a JointTrajectory message from the /set_joint_trajectory topic
-            and move the machine accordingly. It's a bit clunky but it works. -->
-    <!-- You'll probably want to add damping to the joints to stop them it flopping around.
-            e.g. <dynamics damping="10.0" friction="10.0"/> -->
-    <!-- Here's an example message to publish to test it:
-            ros2 topic pub -1 /set_joint_trajectory trajectory_msgs/msg/JointTrajectory  '{header: {frame_id: world}, joint_names: [slider_joint, arm_joint], points: [  {positions: {0.8,0.6}} ]}' -->
-    <!-- Gazebo Parameters -->
-    <gazebo reference="Roue arrière gauche">
-        <mu1>1.0</mu1>
-        <mu2>1.0</mu2>
-    </gazebo>
-    <gazebo reference="Roue arrière droite">
-        <mu1>1.0</mu1>
-        <mu2>1.0</mu2>
-    </gazebo>
-    <gazebo reference="base_link">
-        <mu1>1.0</mu1>
-        <mu2>1.0</mu2>
-    </gazebo>
-    <gazebo reference="Roue avant droite">
-        <mu1>0.00001</mu1>
-        <mu2>0.00001</mu2>
-    </gazebo>
-    <gazebo reference="Roue avant gauche">
-        <mu1>0.00001</mu1>
-        <mu2>0.00001</mu2>
+    <gazebo reference="lidar">
+        <sensor name="laser" type="gpu_lidar">
+            <pose> 0 0 0 0 0 0 </pose>
+            <always_on>true</always_on>
+            <visualize>true</visualize>
+            <update_rate>10</update_rate>
+            <topic>scan</topic>
+            <gz_frame_id>lidar</gz_frame_id>
+            <lidar>
+                <scan>
+                    <horizontal>
+                    <samples>720</samples>
+                    <resolution>1</resolution>
+                    <min_angle>-3.14</min_angle>
+                    <max_angle>3.14</max_angle>
+                    </horizontal>
+                </scan>
+                <range>
+                    <min>0.05</min>
+                    <max>10.0</max>
+                    <resolution>0.01</resolution>
+                </range>
+                <noise>
+                    <type>gaussian</type>
+                    <mean>0.0</mean>
+                    <stddev>0.01</stddev>
+                </noise>
+                <frame_id>lidar</frame_id>
+            </lidar>
+            <always_on>1</always_on>
+            <visualize>true</visualize>
+        </sensor>
     </gazebo>
 </robot>
