Commit message: Manage real robot controller

File: description/lemower.xacro (robot description, xacro)
@@ -2,4 +2,7 @@
 <!-- Description of the LEMOWER robot with XACRO to avoid repeating data -->
 <robot xmlns:xacro="http://www.ros.org/wiki/xacro"  name="lemower">
+    <xacro:arg name="sim_mode" default="false"/>
+    <!-- gestion des parametres -->
+    <xacro:arg name="use_ros2_control" default="true"/>
     <!-- This will include all the contents of example_include.xacro first. Go check it out! -->
     <xacro:include filename="lemower_include.xacro" />
@@ -7,5 +10,10 @@
     <xacro:include filename="lemower_core.xacro" />
     <xacro:include filename="lemower_gazebo.xacro" />
-    <xacro:include filename="ros2_control.xacro"/>
-    <!-- <xacro:include filename="lemower_gz_control.xacro" /> -->
+    <!-- Switch between ros2_control and Gazebo integrated diff-drive control -->
+    <xacro:if value="$(arg use_ros2_control)">
+        <xacro:include filename="ros2_control.xacro" />
+    </xacro:if>
+    <xacro:unless value="$(arg use_ros2_control)">
+        <xacro:include filename="lemower_gz_control.xacro" />
+    </xacro:unless>
 </robot>

File: description/ros2_control.xacro (robot description, xacro)
@@ -1,30 +1,65 @@
 <?xml version="1.0"?>
 <robot xmlns:xacro="http://www.ros.org/wiki/xacro">
-    <ros2_control name="GazeboSystem" type="system">
-        <hardware>
-            <plugin>gz_ros2_control/GazeboSimSystem</plugin>
-        </hardware>
-        <joint name="base_to_roue_arriere_gauche">
+    <xacro:arg name="sim_mode" default="false"/>
+    <xacro:if value="$(arg sim_mode)">
+        <ros2_control name="GazeboSystem" type="system">
+            <hardware>
+                <plugin>gz_ros2_control/GazeboSimSystem</plugin>
+            </hardware>
+            <joint name="base_to_roue_arriere_gauche">
+                <command_interface name="velocity">
+                    <param name="min">-10</param>
+                    <param name="max">10</param>
+                </command_interface>
+            <state_interface name="position"/>
+            <state_interface name="velocity"/>
+            </joint>
+            <joint name="base_to_roue_arriere_droite">
             <command_interface name="velocity">
-                <param name="min">-10</param>
-                <param name="max">10</param>
+                    <param name="min">-10</param>
+                    <param name="max">10</param>
             </command_interface>
-           <state_interface name="position"/>
-           <state_interface name="velocity"/>
-        </joint>
-        <joint name="base_to_roue_arriere_droite">
-           <command_interface name="velocity">
-                <param name="min">-10</param>
-                <param name="max">10</param>
-           </command_interface>
-           <state_interface name="position"/>
-           <state_interface name="velocity"/>
-        </joint>
-    </ros2_control>
-    <gazebo>
-      <plugin filename="gz_ros2_control-system" name="gz_ros2_control::GazeboSimROS2ControlPlugin">
-        <!-- Chemin vers votre fichier de configuration YAML des contrôleurs -->
-        <parameters>$(find lemower_package)/config/my_controllers.yaml</parameters>
-      </plugin>
-    </gazebo>
+            <state_interface name="position"/>
+            <state_interface name="velocity"/>
+            </joint>
+        </ros2_control>
+        <gazebo>
+        <plugin filename="gz_ros2_control-system" name="gz_ros2_control::GazeboSimROS2ControlPlugin">
+            <!-- Chemin vers votre fichier de configuration YAML des contrôleurs -->
+            <parameters>$(find lemower_package)/config/my_controllers.yaml</parameters>
+        </plugin>
+        </gazebo>
+    </xacro:if>
+     <xacro:unless value="$(arg sim_mode)">
+        <!-- Real stuff will go here -->
+        <ros2_control name="RealRobot" type="system">
+            <hardware>
+                <plugin>diffdrive_arduino/DiffDriveArduinoHardware</plugin>
+                <param name="left_wheel_name">left_wheel_joint</param>
+                <param name="right_wheel_name">right_wheel_joint</param>
+                <param name="loop_rate">30</param>
+                <param name="device">/dev/ttyACM0</param>
+                <param name="baud_rate">57600</param>
+                <param name="timeout_ms">1000</param>
+                <param name="enc_counts_per_rev">1440</param>
+            </hardware>
+            <!-- Note everything below here is the same as the Gazebo one -->
+            <joint name="left_wheel_joint">
+                <command_interface name="velocity">
+                    <param name="min">-10</param>
+                    <param name="max">10</param>
+                </command_interface>
+                <state_interface name="position"/>
+                <state_interface name="velocity"/>
+            </joint>
+            <joint name="right_wheel_joint">
+                <command_interface name="velocity">
+                    <param name="min">-10</param>
+                    <param name="max">10</param>
+                </command_interface>
+                <state_interface name="position"/>
+                <state_interface name="velocity"/>
+            </joint>
+        </ros2_control>
+    </xacro:unless>
 </robot>
